Commit message: s

File: Spider_Assembly_fineMesh_frictionDamp/urdf/Spider_Assembly_fineMesh_frictionDamp.urdf (robot description, URDF)
Before this commit: robot Spider_Assembly_fineMesh_frictionDamp, 19 links, 18 joints
Joints:
- joint base_to_coxa1: limit lower=-1.0472 upper=1.0472 effort=10 velocity=10 -> lower=-1.0472 upper=1.0472 effort=0.95 velocity=6
- joint base_to_coxa2: limit lower=-1.0472 upper=1.0472 effort=10 velocity=10 -> lower=-1.0472 upper=1.0472 effort=0.95 velocity=6
- joint base_to_coxa3: limit lower=-1.0472 upper=1.0472 effort=10 velocity=10 -> lower=-1.0472 upper=1.0472 effort=0.95 velocity=6
- joint base_to_coxa4: limit lower=-1.0472 upper=1.0472 effort=10 velocity=10 -> lower=-1.0472 upper=1.0472 effort=0.95 velocity=6
- joint base_to_coxa5: limit lower=-1.0472 upper=1.0472 effort=10 velocity=10 -> lower=-1.0472 upper=1.0472 effort=0.95 velocity=6
- joint base_to_coxa6: limit lower=-1.0472 upper=1.0472 effort=10 velocity=10 -> lower=-1.0472 upper=1.0472 effort=0.95 velocity=6
- joint coxa1_to_femur1: limit lower=-1.5708 upper=2.0944 effort=10 velocity=10 -> lower=-1.0472 upper=1.0472 effort=0.95 velocity=6
- joint coxa2_to_femur2: limit lower=-1.5708 upper=2.0944 effort=10 velocity=10 -> lower=-1.0472 upper=1.0472 effort=0.95 velocity=6
- joint coxa3_to_femur3: limit lower=-1.5708 upper=2.0944 effort=10 velocity=10 -> lower=-1.0472 upper=1.0472 effort=0.95 velocity=6
- joint coxa4_to_femur4: limit lower=-1.5708 upper=2.0944 effort=10 velocity=10 -> lower=-1.0472 upper=1.0472 effort=0.95 velocity=6
- joint coxa5_to_femur5: limit lower=-1.5708 upper=2.0944 effort=10 velocity=10 -> lower=-1.0472 upper=1.0472 effort=0.95 velocity=6
- joint coxa6_to_femur6: limit lower=-1.5708 upper=2.0944 effort=10 velocity=10 -> lower=-1.0472 upper=1.0472 effort=0.95 velocity=6
- joint femur1_to_tibia1: limit lower=-2.0944 upper=1.0472 effort=10 velocity=10 -> lower=-1.0472 upper=1.0472 effort=0.95 velocity=6
- joint femur2_to_tibia2: limit lower=-2.0944 upper=1.0472 effort=10 velocity=10 -> lower=-1.0472 upper=1.0472 effort=0.95 velocity=6
- joint femur3_to_tibia3: limit lower=-2.0944 upper=1.0472 effort=10 velocity=10 -> lower=-1.0472 upper=1.0472 effort=0.95 velocity=6
- joint femur4_to_tibia4: limit lower=-2.0944 upper=1.0472 effort=10 velocity=10 -> lower=-1.0472 upper=1.0472 effort=0.95 velocity=6
- joint femur5_to_tibia5: limit lower=-2.0944 upper=1.0472 effort=10 velocity=10 -> lower=-1.0472 upper=1.0472 effort=0.95 velocity=6
- joint femur6_to_tibia6: limit lower=-2.0944 upper=1.0472 effort=10 velocity=10 -> lower=-1.0472 upper=1.0472 effort=0.95 velocity=6
